Commit message: test

File: tmp/rf2502_new_3.urdf (robot description, URDF)
Before this commit: robot rf2502_new_3, 21 links, 20 joints
Links:
- link arml_Link: geometry collision mesh filename=package://rf2502_new_3/meshes/arml_Link.STL; visual mesh filename=package://rf2502_new_3/meshes/arml_Link.STL
- link arml_Link1: geometry collision mesh filename=package://rf2502_new_3/meshes/arml_Link1.STL; visual mesh filename=package://rf2502_new_3/meshes/arml_Link1.STL
- link arml_Link2: geometry collision mesh filename=package://rf2502_new_3/meshes/arml_Link2.STL; visual mesh filename=package://rf2502_new_3/meshes/arml_Link2.STL
- link arml_Link3: geometry collision mesh filename=package://rf2502_new_3/meshes/arml_Link3.STL; visual mesh filename=package://rf2502_new_3/meshes/arml_Link3.STL
- link arml_Link4: geometry collision mesh filename=package://rf2502_new_3/meshes/arml_Link4.STL; visual mesh filename=package://rf2502_new_3/meshes/arml_Link4.STL
- link arml_Link5: geometry collision mesh filename=package://rf2502_new_3/meshes/arml_Link5.STL; visual mesh filename=package://rf2502_new_3/meshes/arml_Link5.STL
- link armr_Link: geometry collision mesh filename=package://rf2502_new_3/meshes/armr_Link.STL; visual mesh filename=package://rf2502_new_3/meshes/armr_Link.STL
- link armr_Link1: geometry collision mesh filename=package://rf2502_new_3/meshes/armr_Link1.STL; visual mesh filename=package://rf2502_new_3/meshes/armr_Link1.STL
- link armr_Link2: geometry collision mesh filename=package://rf2502_new_3/meshes/armr_Link2.STL; visual mesh filename=package://rf2502_new_3/meshes/armr_Link2.STL
- link armr_Link3: geometry collision mesh filename=package://rf2502_new_3/meshes/armr_Link3.STL; visual mesh filename=package://rf2502_new_3/meshes/armr_Link3.STL
- link armr_Link4: geometry collision mesh filename=package://rf2502_new_3/meshes/armr_Link4.STL; visual mesh filename=package://rf2502_new_3/meshes/armr_Link4.STL
- link armr_Link5: geometry collision mesh filename=package://rf2502_new_3/meshes/armr_Link5.STL; visual mesh filename=package://rf2502_new_3/meshes/armr_Link5.STL
- link base_link: geometry collision mesh filename=package://rf2502_new_3/meshes/base_link.STL; visual mesh filename=package://rf2502_new_3/meshes/base_link.STL
- link body_Link1: geometry collision mesh filename=package://rf2502_new_3/meshes/body_Link1.STL; visual mesh filename=package://rf2502_new_3/meshes/body_Link1.STL
- link body_Link2: geometry collision mesh filename=package://rf2502_new_3/meshes/body_Link2.STL; visual mesh filename=package://rf2502_new_3/meshes/body_Link2.STL
- link body_Link3: geometry collision mesh filename=package://rf2502_new_3/meshes/body_Link3.STL; visual mesh filename=package://rf2502_new_3/meshes/body_Link3.STL
- link body_Link4: geometry collision mesh filename=package://rf2502_new_3/meshes/body_Link4.STL; visual mesh filename=package://rf2502_new_3/meshes/body_Link4.STL
- link handl_Link1: geometry collision mesh filename=package://rf2502_new_3/meshes/handl_Link1.STL; visual mesh filename=package://rf2502_new_3/meshes/handl_Link1.STL
- link handl_Link2: geometry collision mesh filename=package://rf2502_new_3/meshes/handl_Link2.STL; visual mesh filename=package://rf2502_new_3/meshes/handl_Link2.STL
- link handr_Link1: geometry collision mesh filename=package://rf2502_new_3/meshes/handr_Link1.STL; visual mesh filename=package://rf2502_new_3/meshes/handr_Link1.STL
- link handr_Link2: geometry collision mesh filename=package://rf2502_new_3/meshes/handr_Link2.STL; visual mesh filename=package://rf2502_new_3/meshes/handr_Link2.STL
Joints:
- joint body_joint1: origin xyz=0 0.689 0.12151 rpy=0 0 0 -> xyz=0 -0.12151 0.689 rpy=1.5708 0 0
